File: 2Moons PCB/Kyuu.sch (KiCad schematic (older format))
At the start: 152 parts, among them K0 KEYSW, K1 KEYSW, K10 KEYSW, K11 KEYSW, K12 KEYSW, K13 KEYSW, K13_1 KEYSW, K14 KEYSW, K15 KEYSW, K16 KEYSW, K17 KEYSW, K18 KEYSW, K19 KEYSW, K2 KEYSW, K20 KEYSW, K21 KEYSW, K22 KEYSW, K23 KEYSW, K24 KEYSW, K25 KEYSW, K26 KEYSW, K27 KEYSW, K28 KEYSW, K29 KEYSW, K29_1 KEYSW, K3 KEYSW, K30 KEYSW, K31 KEYSW, K32 KEYSW, K33 KEYSW, K34 KEYSW, K35 KEYSW, K36 KEYSW, K37 KEYSW, K38 KEYSW, K39 KEYSW, K4 KEYSW, K40 KEYSW, K41 KEYSW, K42 KEYSW, K43 KEYSW, K44 KEYSW, K45 KEYSW, K46 KEYSW, K47 KEYSW, K48 KEYSW, K49 KEYSW, K5 KEYSW, K50 KEYSW, K51 KEYSW, K52 KEYSW, K53 KEYSW, K54 KEYSW, K55 KEYSW, K56 KEYSW, K57 KEYSW, K58 KEYSW, K59 KEYSW, K6 KEYSW, K60 KEYSW, K61 KEYSW, K62 KEYSW, K63 KEYSW, K64 KEYSW, K7 KEYSW, K8 KEYSW, K9 KEYSW, SW1 SW_PUSH, U1 ATMEGA32U4, X1 XTAL_GND

Commit message: PCB with ESD Added
Parts:
- added F1: 500mA, Fuse:Fuse_1206_3216Metric, symbol device:Polyfuse_Small
- added U2: SRV05-4, Package_TO_SOT_SMD:SOT-23-6_Handsoldering, symbol ESD_Protection:SRV05-4
- C1, C2, C3, C4, C6: LCSC Part# (none) -> C14663; Mrf (none) -> YAGEO; Part# (none) -> CC0603KRX7R9BB104
- C5: LCSC Part# (none) -> C19666; Mrf (none) -> Samsung Electro-Mechanics; Part# (none) -> CL10A475KO8NNNC
- C7, C8: value C_Small -> 18pF; LCSC Part# (none) -> C1647; Mrf (none) -> Samsung Electro-Mechanics; Part# (none) -> CL10C180JB8NNNC
- D1, D10, D11, D12, D13, D14, D15, D16, D17, D18, D19, D2, D20, D21, D22, D24, D25, D26, D27, D28, D29, D3, D30, D31, D32, D33, D34, D35, D36, D37, D38, D39, D4, D40, D41, D42, D43, D44, D45, D46, D47, D48, D49, D5, D50, D51, D52, D53, D54, D55, D56, D57, D58, D59, D6, D60, D61, D62, D63, D64, D65, D66, D7, D8, D9: LCSC Part# (none) -> C81598; Mrf (none) -> Semtech; Part# (none) -> 1N4148W
- D23: Datasheet (none) -> https://datasheet.lcsc.com/szlcsc/Semtech-1N4148W_C81598.pdf; LCSC Part# (none) -> C81598; Mrf (none) -> Semtech; Part# (none) -> 1N4148W
- R1, R2: value 5.5k -> 5.1k; LCSC Part# (none) -> C23186; Mfr (none) -> Uniroyal Elec; Part# (none) -> 0603WAF5101T5E
- R3, R4: LCSC Part# (none) -> C23345; Mrf (none) -> Uniroyal Elec; Part# (none) -> 0603WAF220JT5E
- R5, R6: LCSC Part# (none) -> C25804; Mrf (none) -> Uniroyal Elec; Part# (none) -> 0603WAF1002T5E
- SW1: LCSC Part# (none) -> C221929; Mrf (none) -> C&K; Part# (none) -> RS-187R05A2-DSMTRT
- U1: LCSC Part# (none) -> C44854; Mrf (none) -> Microchip Tech; Part# (none) -> ATMEGA32U4-AU
- USB1: footprint (none) -> Type-C:HRO-TYPE-C-31-M-12-HandSoldering; LCSC Part# (none) -> C165948; Mrf (none) -> Korean Hroparts Elec; Part# (none) -> TYPE-C-31-M-12
- X1: LCSC Part# (none) -> C164044; Mrf (none) -> Zhejiang Abel Elec; Part# (none) -> TAXM16M4RDBCCT2T
Connections:
- net D+: now also U2.6 (IO4)
- net D-: now also U2.1 (IO1)
- net GND: now also USB1.12 (GND), USB1.13 (SHIELD), U2.2 (VN)
- net VCC: now also USB1.11 (VBUS), F1.2, U2.5 (VP); no longer C1.2, C2.2, C3.2, C4.2, C5.2, R5.1, U1.14 (VCC), U1.2 (UVcc), U1.24 (AVCC), U1.34 (VCC), U1.44 (AVCC), U1.7 (VBus)
- new net +5V: C1.2, C2.2, C3.2, C4.2, C5.2, F1.1, R5.1, U1.14 (VCC), U1.2 (UVcc), U1.24 (AVCC), U1.34 (VCC), U1.44 (AVCC), U1.7 (VBus)
- no-connect marks 3 -> 2

Commit message: Kyuu New PCB
Parts:
- F1: symbol device:Polyfuse_Small -> Kyuu-rescue:Polyfuse_Small-device
- U2: symbol ESD_Protection:SRV05-4 -> Kyuu-rescue:SRV05-4-ESD_Protection
Changed lines of the file:
@@
 	3450 6850 4350 6850
 $Comp
-L ESD_Protection:SRV05-4 U2
+L Kyuu-rescue:SRV05-4-ESD_Protection U2
 U 1 1 5FD0EDC3
 P 6650 8325
@@
 	4500 9150 5500 9150
 $Comp
-L device:Polyfuse_Small F1
+L Kyuu-rescue:Polyfuse_Small-device F1
 U 1 1 60020D25
 P 5775 8750
